Commit message: added ur5_gripper.urdf

File: urdf/ur5_gripper.urdf (robot description, URDF)
Before this commit: robot sisbot, 19 links, 18 joints
Links:
- removed link robotiq_85_adapter_link
- removed link robotiq_85_base_link
- removed link robotiq_85_left_finger_link
- removed link robotiq_85_left_finger_tip_link
- removed link robotiq_85_left_inner_knuckle_link
- removed link robotiq_85_left_knuckle_link
- removed link robotiq_85_right_finger_link
- removed link robotiq_85_right_finger_tip_link
- removed link robotiq_85_right_inner_knuckle_link
- removed link robotiq_85_right_knuckle_link
- link base_link: geometry collision mesh filename=../meshes/ur5/collision/base.stl; visual mesh filename=../meshes/ur5/visual/base.obj
- link forearm_link: mass 0 -> 2.275; geometry collision mesh filename=../meshes/ur5/collision/forearm.stl; visual mesh filename=../meshes/ur5/visual/forearm.obj
- link shoulder_link: geometry collision mesh filename=../meshes/ur5/collision/shoulder.stl; visual mesh filename=../meshes/ur5/visual/shoulder.obj
- link upper_arm_link: mass 0 -> 8.393; geometry collision mesh filename=../meshes/ur5/collision/upperarm.stl; visual mesh filename=../meshes/ur5/visual/upperarm.obj
- link wrist_1_link: mass 0 -> 1.219; geometry collision mesh filename=../meshes/ur5/collision/wrist1.stl; visual mesh filename=../meshes/ur5/visual/wrist1.obj
- link wrist_2_link: mass 0 -> 1.219; geometry collision mesh filename=../meshes/ur5/collision/wrist2.stl; visual mesh filename=../meshes/ur5/visual/wrist2.obj
- link wrist_3_link: mass 0 -> 0.1879; geometry collision mesh filename=../meshes/ur5/collision/wrist3.stl; visual mesh filename=../meshes/ur5/visual/wrist3.obj
Joints:
- removed joint arm_gripper_joint
- removed joint robotiq_85_base_joint
- removed joint robotiq_85_left_finger_joint
- removed joint robotiq_85_left_finger_tip_joint
- removed joint robotiq_85_left_inner_knuckle_joint
- removed joint robotiq_85_left_knuckle_joint
- removed joint robotiq_85_right_finger_joint
- removed joint robotiq_85_right_finger_tip_joint
- removed joint robotiq_85_right_inner_knuckle_joint
- removed joint robotiq_85_right_knuckle_joint
- joint elbow_joint: limit lower=-3.14159265359 upper=3.14159265359 effort=150.0 velocity=3.15 -> lower=-3.14159265359 upper=3.14159265359 effort=300.0 velocity=10
- joint shoulder_lift_joint: limit lower=-3.14159265359 upper=3.14159265359 effort=150.0 velocity=3.15 -> lower=-3.14159265359 upper=3.14159265359 effort=300.0 velocity=10; origin xyz=0.0 0.13585 0.0 rpy=0.0 1.57079632679 0.0 -> xyz=0.0 0.13585 0.0 rpy=0.0 4.8 0.0
- joint shoulder_pan_joint: limit lower=-3.14159265359 upper=3.14159265359 effort=150.0 velocity=3.15 -> lower=-3.14159265359 upper=3.14159265359 effort=300.0 velocity=10; origin xyz=0.0 0.0 0.089159 rpy=0.0 0.0 0.0 -> xyz=0.0 0.0 0.089159 rpy=0.0 0.0 3.14
- joint world_joint: origin xyz=0.0 0.0 0.1 rpy=0.0 0.0 -0.6 -> xyz=0.0 0.0 0.1 rpy=0.0 0.0 0
- joint wrist_1_joint: limit lower=-3.14159265359 upper=3.14159265359 effort=28.0 velocity=3.2 -> lower=-3.14159265359 upper=3.14159265359 effort=300.0 velocity=10
- joint wrist_2_joint: limit lower=-3.14159265359 upper=3.14159265359 effort=28.0 velocity=3.2 -> lower=-3.14159265359 upper=3.14159265359 effort=300.0 velocity=10
- joint wrist_3_joint: limit lower=-3.14159265359 upper=3.14159265359 effort=28.0 velocity=3.2 -> lower=-3.14159265359 upper=3.14159265359 effort=300.0 velocity=10

Commit message: added robotiq_2f_85 gripper files

File: urdf/ur5_gripper.urdf (robot description, URDF)
Before this commit: robot universal_robot, 9 links, 8 joints
Links:
- added link robotiq_85_adapter_link; collision mesh filename=../meshes/robotiq_c2/collision/robotiq_85_gripper_adapter_p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; visual mesh filename=../meshes/robotiq_c2/visual/robotiq_85_gripper_adapter_plat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
- added link robotiq_85_base_link; collision mesh filename=../meshes/robotiq_c2/collision/robotiq_85_gripper_base.stl; visual mesh filename=../meshes/robotiq_c2/visual/robotiq_85_gripper_base.obj
- added link robotiq_85_left_finger_link; collision mesh filename=../meshes/robotiq_c2/collision/robotiq_85_gripper_joint_1_L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; visual mesh filename=../meshes/robotiq_c2/visual/robotiq_85_gripper_joint_1_L.obj
- added link robotiq_85_left_finger_tip_link; collision mesh filename=../meshes/robotiq_c2/collision/robotiq_85_gripper_joint_3_L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; visual mesh filename=../meshes/robotiq_c2/visual/robotiq_85_gripper_joint_3_L.obj
- added link robotiq_85_left_inner_knuckle_link; collision mesh filename=../meshes/robotiq_c2/collision/robotiq_85_gripper_joint_2_L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; visual mesh filename=../meshes/robotiq_c2/visual/robotiq_85_gripper_joint_2_L.obj
- added link robotiq_85_left_knuckle_link; collision mesh filename=../meshes/robotiq_c2/collision/robotiq_85_gripper_joint_0_L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; visual mesh filename=../meshes/robotiq_c2/visual/robotiq_85_gripper_joint_0_L.obj
- added link robotiq_85_right_finger_link; collision mesh filename=../meshes/robotiq_c2/collision/robotiq_85_gripper_joint_1_R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; visual mesh filename=../meshes/robotiq_c2/visual/robotiq_85_gripper_joint_1_R.obj
- added link robotiq_85_right_finger_tip_link; collision mesh filename=../meshes/robotiq_c2/collision/robotiq_85_gripper_joint_3_R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; visual mesh filename=../meshes/robotiq_c2/visual/robotiq_85_gripper_joint_3_R.obj
- added link robotiq_85_right_inner_knuckle_link; collision mesh filename=../meshes/robotiq_c2/collision/robotiq_85_gripper_joint_2_R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; visual mesh filename=../meshes/robotiq_c2/visual/robotiq_85_gripper_joint_2_R.obj
- added link robotiq_85_right_knuckle_link; collision mesh filename=../meshes/robotiq_c2/collision/robotiq_85_gripper_joint_0_R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; visual mesh filename=../meshes/robotiq_c2/visual/robotiq_85_gripper_joint_0_R.obj
Joints:
- added joint robotiq_85_base_joint: type fixed, parent robotiq_85_adapter_link, child robotiq_85_base_link, origin xyz=.0085 0 -.0041 rpy=0 0 0, axis 1 0 0
- added joint robotiq_85_left_finger_joint: type fixed, parent robotiq_85_left_knuckle_link, child robotiq_85_left_finger_link, origin xyz=0 .00508 .03134 rpy=6.1415 0 0, axis 1 0 0, limit lower=0 upper=1.5707 effort=1000 velocity=2.0
- added joint robotiq_85_left_finger_tip_joint: type revolute, parent robotiq_85_left_inner_knuckle_link, child robotiq_85_left_finger_tip_link, origin xyz=0 .04196 -.0388 rpy=0 0 0, axis 1 0 0, limit lower=0 upper=1.5707 effort=1000 velocity=2.0, mimic joint=robotiq_85_left_knuckle_joint multiplier=-1
- added joint robotiq_85_left_inner_knuckle_joint: type revolute, parent robotiq_85_base_link, child robotiq_85_left_inner_knuckle_link, origin xyz=.04843 .0127 0 rpy=1.5707 1.5707 0, axis 1 0 0, limit lower=0 upper=1.5707 effort=1000 velocity=2.0, mimic joint=robotiq_85_left_knuckle_joint offset=0
- added joint robotiq_85_left_knuckle_joint: type revolute, parent robotiq_85_base_link, child robotiq_85_left_knuckle_link, origin xyz=0.04191 0.0306 0 rpy=-1.5707 1.5707 0, axis 1 0 0, limit lower=0 upper=0.343 effort=1000 velocity=2.0
- added joint robotiq_85_right_finger_joint: type fixed, parent robotiq_85_right_knuckle_link, child robotiq_85_right_finger_link, origin xyz=0 .00508 .03134 rpy=6.1415 0 0, axis 1 0 0, limit lower=0 upper=1.5707 effort=1000 velocity=2.0
- added joint robotiq_85_right_finger_tip_joint: type revolute, parent robotiq_85_right_inner_knuckle_link, child robotiq_85_right_finger_tip_link, origin xyz=0 .04196 -.0388 rpy=0 0 0, axis 1 0 0, limit lower=0 upper=1.5707 effort=1000 velocity=2.0, mimic joint=robotiq_85_left_knuckle_joint multiplier=-1
- added joint robotiq_85_right_inner_knuckle_joint: type revolute, parent robotiq_85_base_link, child robotiq_85_right_inner_knuckle_link, origin xyz=.04843 -.0127 0 rpy=-1.5707 -1.5707 0, axis 1 0 0, limit lower=0 upper=1.5707 effort=1000 velocity=2.0, mimic joint=robotiq_85_left_knuckle_joint offset=0
- added joint robotiq_85_right_knuckle_joint: type revolute, parent robotiq_85_base_link, child robotiq_85_right_knuckle_link, origin xyz=.04191 -.0306 0 rpy=1.5707 -1.5707 0, axis 1 0 0, limit lower=0 upper=1.5707 effort=1000 velocity=2.0, mimic joint=robotiq_85_left_knuckle_joint multiplier=1
