Commit message: updated gripper urdf and meshes, found out pybullet uses only last material in urdf

File: urdf/gripper.urdf (robot description, URDF)
Before this commit: robot robotiq_c2, 11 links, 10 joints
Links:
- removed link robotiq_85_adapter_link
- removed link robotiq_85_left_finger_link
- removed link robotiq_85_left_finger_tip_link
- removed link robotiq_85_left_inner_knuckle_link
- removed link robotiq_85_left_knuckle_link
- removed link robotiq_85_right_finger_link
- removed link robotiq_85_right_finger_tip_link
- removed link robotiq_85_right_inner_knuckle_link
- removed link robotiq_85_right_knuckle_link
- removed link world
- link robotiq_85_base_link: mass None -> 0.30915; geometry collision mesh filename=/home/sudhir/robotics/git_hub_repos/pick-place-robot/meshes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 scale=0.005 0.005 0.005; visual mesh filename=/home/sudhir/robotics/git_hub_repos/pick-place-robot/meshes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 scale=0.005 0.005 0.005
Joints:
- removed joint robotiq_85_base_joint
- removed joint robotiq_85_left_finger_joint
- removed joint robotiq_85_left_finger_tip_joint
- removed joint robotiq_85_left_inner_knuckle_joint
- removed joint robotiq_85_left_knuckle_joint
- removed joint robotiq_85_right_finger_joint
- removed joint robotiq_85_right_finger_tip_joint
- removed joint robotiq_85_right_inner_knuckle_joint
- removed joint robotiq_85_right_knuckle_joint
- removed joint world_joint
