Commit message: updated urdf and meshes files and cleanup

File: urdf/robotiq_2f_85.urdf (robot description, URDF)
Before this commit: robot robotiq_arg85_description, 9 links, 8 joints
Links:
- link left_inner_finger: geometry collision mesh filename=../meshes/robotiq_2f_85/collision/inner_finger_coarse.STL; visual mesh filename=../meshes/robotiq_2f_85/visual/inner_finger_fine.STL
- link left_inner_knuckle: geometry collision mesh filename=../meshes/robotiq_2f_85/collision/inner_knuckle_coarse.STL; visual mesh filename=../meshes/robotiq_2f_85/visual/inner_knuckle_fine.STL
- link left_outer_finger: geometry collision mesh filename=../meshes/robotiq_2f_85/collision/outer_finger_coarse.STL; visual mesh filename=../meshes/robotiq_2f_85/visual/outer_finger_fine.STL
- link left_outer_knuckle: geometry collision mesh filename=../meshes/robotiq_2f_85/collision/outer_knuckle_coarse.STL; visual mesh filename=../meshes/robotiq_2f_85/visual/outer_knuckle_fine.STL
- link right_inner_finger: geometry collision mesh filename=../meshes/robotiq_2f_85/collision/inner_finger_coarse.STL; visual mesh filename=../meshes/robotiq_2f_85/visual/inner_finger_fine.STL
- link right_inner_knuckle: geometry collision mesh filename=../meshes/robotiq_2f_85/collision/inner_knuckle_coarse.STL; visual mesh filename=../meshes/robotiq_2f_85/visual/inner_knuckle_fine.STL
- link right_outer_finger: geometry collision mesh filename=../meshes/robotiq_2f_85/collision/outer_finger_coarse.STL; visual mesh filename=../meshes/robotiq_2f_85/visual/outer_finger_fine.STL
- link right_outer_knuckle: geometry collision mesh filename=../meshes/robotiq_2f_85/collision/outer_knuckle_coarse.STL; visual mesh filename=../meshes/robotiq_2f_85/visual/outer_knuckle_fine.STL
- link robotiq_85_base_link: geometry collision mesh filename=../meshes/robotiq_2f_85/collision/robotiq_85_base_link_coar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; visual mesh filename=../meshes/robotiq_2f_85/visual/robotiq_85_base_link_fine.STL

File: urdf/robotiq_2f_85_actual_mesh.urdf (robot description, URDF)
Before this commit: robot robotiq_arg85_description, 9 links, 8 joints
Links:
- link left_inner_finger: geometry collision mesh filename=../meshes/robotiq_2f_85_original/collision/robotiq_arg2f_85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 scale=0.001 0.001 0.001; visual mesh filename=../meshes/robotiq_2f_85_original/visual/robotiq_arg2f_85_in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 scale=0.001 0.001 0.001
- link left_inner_knuckle: geometry collision mesh filename=../meshes/robotiq_2f_85_original/collision/robotiq_arg2f_85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 scale=0.001 0.001 0.001; visual mesh filename=../meshes/robotiq_2f_85_original/visual/robotiq_arg2f_85_in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 scale=0.001 0.001 0.001
- link left_outer_finger: geometry collision mesh filename=../meshes/robotiq_2f_85_original/collision/robotiq_arg2f_85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 scale=0.001 0.001 0.001; visual mesh filename=../meshes/robotiq_2f_85_original/visual/robotiq_arg2f_85_ou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 scale=0.001 0.001 0.001
- link left_outer_knuckle: geometry collision mesh filename=../meshes/robotiq_2f_85_original/collision/robotiq_arg2f_85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 scale=0.001 0.001 0.001; visual mesh filename=../meshes/robotiq_2f_85_original/visual/robotiq_arg2f_85_ou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 scale=0.001 0.001 0.001
- link right_inner_finger: geometry collision mesh filename=../meshes/robotiq_2f_85_original/collision/robotiq_arg2f_85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 scale=0.001 0.001 0.001; visual mesh filename=../meshes/robotiq_2f_85_original/visual/robotiq_arg2f_85_in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 scale=0.001 0.001 0.001
- link right_inner_knuckle: geometry collision mesh filename=../meshes/robotiq_2f_85_original/collision/robotiq_arg2f_85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 scale=0.001 0.001 0.001; visual mesh filename=../meshes/robotiq_2f_85_original/visual/robotiq_arg2f_85_in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 scale=0.001 0.001 0.001
- link right_outer_finger: geometry collision mesh filename=../meshes/robotiq_2f_85_original/collision/robotiq_arg2f_85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; visual mesh filename=../meshes/robotiq_2f_85_original/visual/robotiq_arg2f_85_ou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 scale=0.001 0.001 0.001
- link right_outer_knuckle: geometry collision mesh filename=../meshes/robotiq_2f_85_original/collision/robotiq_arg2f_85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 scale=0.001 0.001 0.001; visual mesh filename=../meshes/robotiq_2f_85_original/visual/robotiq_arg2f_85_ou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 scale=0.001 0.001 0.001
- link robotiq_85_base_link: geometry collision mesh filename=../meshes/robotiq_2f_85_original/collision/robotiq_arg2f_85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 scale=0.001 0.001 0.001; visual mesh filename=../meshes/robotiq_2f_85_original/visual/robotiq_arg2f_85_ba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 scale=0.001 0.001 0.001

File: urdf/ur5_gripper.urdf (robot description, URDF)
Before this commit: robot universal_robot, 19 links, 17 joints
Links:
- removed link robotiq_85_adapter_link
- removed link robotiq_85_base_link
- removed link robotiq_85_left_finger_link
- removed link robotiq_85_left_finger_tip_link
- removed link robotiq_85_left_inner_knuckle_link
- removed link robotiq_85_left_knuckle_link
- removed link robotiq_85_right_finger_link
- removed link robotiq_85_right_finger_tip_link
- removed link robotiq_85_right_inner_knuckle_link
- removed link robotiq_85_right_knuckle_link
Joints:
- removed joint robotiq_85_base_joint
- removed joint robotiq_85_left_finger_joint
- removed joint robotiq_85_left_finger_tip_joint
- removed joint robotiq_85_left_inner_knuckle_joint
- removed joint robotiq_85_left_knuckle_joint
- removed joint robotiq_85_right_finger_joint
- removed joint robotiq_85_right_finger_tip_joint
- removed joint robotiq_85_right_inner_knuckle_joint
- removed joint robotiq_85_right_knuckle_joint
